Commit message: feat: 迁移 AGV 工程代码，包含所有功能包及 SDK 依赖

File: src/agv_description/urdf/agv.xacro (robot description, xacro)
@@ -262,5 +262,5 @@
     <axis
       xyz="0 0 1" />
-    <limit effort = "1000.0" velocity = "1.0" lower = "-3.14" upper = "3.14"/>
+    <limit effort = "1000.0" velocity = "1.0" lower = "-3.0" upper = "3.0"/>
   </joint>
   <link
@@ -316,5 +316,5 @@
     <axis
       xyz="0 0 1" />
-    <limit effort = "1000.0" velocity = "1.0" lower = "-3.14" upper = "3.14"/>
+    <limit effort = "1000.0" velocity = "1.0" lower = "-3.0" upper = "3.0"/>
   </joint>
   <link
@@ -370,5 +370,5 @@
     <axis
       xyz="0 0 -1" />
-    <limit effort = "1000.0" velocity = "1.0" lower = "-3.14" upper = "3.14"/>
+    <limit effort = "1000.0" velocity = "1.0" lower = "-3.0" upper = "3.0"/>
   </joint>
   <link
@@ -424,5 +424,5 @@
     <axis
       xyz="0 0 1" />
-    <limit effort = "1000.0" velocity = "1.0" lower = "-3.14" upper = "3.14"/>
+    <limit effort = "1000.0" velocity = "1.0" lower = "-3.0" upper = "3.0"/>
   </joint>
   <link
@@ -478,5 +478,5 @@
     <axis
       xyz="0 0 -1" />
-    <limit effort = "1000.0" velocity = "1.0" lower = "-3.14" upper = "3.14"/>
+    <limit effort = "1000.0" velocity = "1.0" lower = "-3.0" upper = "3.0"/>
   </joint>
   <link
@@ -532,5 +532,5 @@
     <axis
       xyz="0 0 1" />
-    <limit effort = "1000.0" velocity = "1.0" lower = "-3.14" upper = "3.14"/>
+    <limit effort = "1000.0" velocity = "1.0" lower = "-3.0" upper = "3.0"/>
   </joint>
   <link
@@ -543,4 +543,12 @@
   </joint>
   <!-- arm2 description-->
+  <link
+    name="arm2_cartesionbase_link" />
+  <joint
+    name="arm2_cartesionbase_joint" type="fixed">
+      <parent link="revolute_link" />
+      <child link="arm2_cartesionbase_link" />
+      <origin xyz="-0.00033177 -0.099999 0.34041" rpy="0 0 1.5708" />
+  </joint>
   <link
     name="arm2_base">
@@ -562,5 +570,5 @@
       <origin
         xyz="0 0 0"
-        rpy="0 0 0" />
+        rpy="0 0 -1.5708" />
       <geometry>
         <mesh
@@ -576,5 +584,5 @@
       <origin
         xyz="0 0 0"
-        rpy="0 0 0" />
+        rpy="0 0 -1.5708" />
       <geometry>
         <mesh
@@ -587,8 +595,11 @@
     type="fixed">
     <origin
+      xyz="0 0 0"
+      rpy="0 -1.5708 0" />
+       <!-- <origin
       xyz="-0.00033177 -0.099999 0.34041"
-      rpy="1.5708 0 -0.0033177" />
-    <parent
-      link="revolute_link" />
+      rpy="0 0 1.5708" /> -->
+    <parent
+      link="arm2_cartesionbase_link" />
     <child
       link="arm2_base" />
@@ -615,5 +626,5 @@
       <origin
         xyz="0 0 0"
-        rpy="0 0 0" />
+        rpy="0 0 -1.5708" />
       <geometry>
         <mesh
@@ -629,5 +640,5 @@
       <origin
         xyz="0 0 0"
-        rpy="0 0 0" />
+        rpy="0 0 -1.5708" />
       <geometry>
         <mesh
@@ -648,5 +659,5 @@
     <axis
       xyz="0 0 1" />
-    <limit effort = "1000.0" velocity = "1.0" lower = "-3.14" upper = "3.14"/>
+    <limit effort = "1000.0" velocity = "1.0" lower = "-3.0" upper = "3.0"/>
   </joint>
   <link
@@ -669,5 +680,5 @@
       <origin
         xyz="0 0 0"
-        rpy="0 0 0" />
+        rpy="-1.5708 -1.5708 0" />
       <geometry>
         <mesh
@@ -683,5 +694,5 @@
       <origin
         xyz="0 0 0"
-        rpy="0 0 0" />
+        rpy="-1.5708 -1.5708 0" />
       <geometry>
         <mesh
@@ -693,7 +704,11 @@
     name="arm2_joint2"
     type="revolute">
-    <origin
+    <!-- <origin
       xyz="-0.0865 0 0.171"
-      rpy="3.1416 -1.5708 3.1416" />
+      rpy="0 0 0" /> -->
+    <origin
+      xyz="0 0.0865 0.171"
+      rpy="0 0 0" />
+      <!-- rpy="3.1416 -1.5708 3.1416" -->
     <parent
       link="arm2_joint1" />
@@ -701,6 +716,6 @@
       link="arm2_joint2" />
     <axis
-      xyz="0 0 1" />
-    <limit effort = "1000.0" velocity = "1.0" lower = "-3.14" upper = "3.14"/>
+      xyz="0 1 0" />
+    <limit effort = "1000.0" velocity = "1.0" lower = "-3.0" upper = "3.0"/>
   </joint>
   <link
@@ -723,5 +738,5 @@
       <origin
         xyz="0 0 0"
-        rpy="0 0 0" />
+        rpy="-1.5708 -1.5708 0" />
       <geometry>
         <mesh
@@ -737,5 +752,5 @@
       <origin
         xyz="0 0 0"
-        rpy="0 0 0" />
+        rpy="-1.5708 -1.5708 0" />
       <geometry>
         <mesh
@@ -748,6 +763,9 @@
     type="revolute">
     <origin
+      xyz="0 0 0.49"
+      rpy="0 0 0" />
+       <!-- <origin
       xyz="0.49 0 0.01"
-      rpy="0 0 0" />
+      rpy="0 0 0" /> -->
     <parent
       link="arm2_joint2" />
@@ -755,6 +773,6 @@
       link="arm2_joint3" />
     <axis
-      xyz="0 0 1" />
-    <limit effort = "1000.0" velocity = "1.0" lower = "-3.14" upper = "3.14"/>
+      xyz="0 -1 0" />
+    <limit effort = "1000.0" velocity = "1.0" lower = "-3.0" upper = "3.0"/>
   </joint>
   <link
@@ -777,5 +795,5 @@
       <origin
         xyz="0 0 0"
-        rpy="0 0 0" />
+        rpy="0 0 -1.5708" />
       <geometry>
         <mesh
@@ -791,5 +809,5 @@
       <origin
         xyz="0 0 0"
-        rpy="0 0 0" />
+        rpy="0 0 -1.5708 "/>
       <geometry>
         <mesh
@@ -802,6 +820,9 @@
     type="revolute">
     <origin
+      xyz="0 -0.0915  0.1475"
+      rpy="0 0 0" />
+       <!-- <origin
       xyz="0.1475 0 -0.0915"
-      rpy="0 1.5708 0" />
+      rpy="0 1.5708 0" /> -->
     <parent
       link="arm2_joint3" />
@@ -810,5 +831,5 @@
     <axis
       xyz="0 0 1" />
-    <limit effort = "1000.0" velocity = "1.0" lower = "-3.14" upper = "3.14"/>
+    <limit effort = "1000.0" velocity = "1.0" lower = "-3.0" upper = "3.0"/>
   </joint>
   <link
@@ -831,5 +852,5 @@
       <origin
         xyz="0 0 0"
-        rpy="0 0 0" />
+        rpy="-1.5708 -1.5708 0" />
       <geometry>
         <mesh
@@ -843,7 +864,7 @@
     </visual>
     <collision>
-      <origin
-        xyz="0 0 0"
-        rpy="0 0 0" />
+    <origin
+        xyz="0 0 0"
+        rpy="-1.5708 -1.5708 0" />
       <geometry>
         <mesh
@@ -855,7 +876,10 @@
     name="arm2_joint5"
     type="revolute">
-    <origin
+    <!-- <origin
       xyz="0.0737 0 0.2125"
-      rpy="3.1416 -1.5708 3.1416" />
+      rpy="3.1416 -1.5708 3.1416" /> -->
+    <origin
+      xyz="0 -0.0737  0.2125"
+      rpy="0 0 0" />
     <parent
       link="arm2_joint4" />
@@ -863,6 +887,6 @@
       link="arm2_joint5" />
     <axis
-      xyz="0 0 1" />
-    <limit effort = "1000.0" velocity = "1.0" lower = "-3.14" upper = "3.14"/>
+      xyz="0 -1 0" />
+    <limit effort = "1000.0" velocity = "1.0" lower = "-3.0" upper = "3.0"/>
   </joint>
   <link
@@ -885,5 +909,5 @@
       <origin
         xyz="0 0 0"
-        rpy="0 0 0" />
+        rpy="0 0 -1.5708" />
       <geometry>
         <mesh
@@ -899,5 +923,5 @@
       <origin
         xyz="0 0 0"
-        rpy="0 0 0" />
+        rpy="0 0 -1.5708" />
       <geometry>
         <mesh
@@ -910,6 +934,9 @@
     type="revolute">
     <origin
+      xyz="0 -0.073  0.0763"
+      rpy="0 0 0" />
+        <!-- <origin
       xyz="0.073 0 -0.0763"
-      rpy="0 1.5708 0" />
+      rpy="0 1.5708 0" /> -->
     <parent
       link="arm2_joint5" />
@@ -918,8 +945,22 @@
     <axis
       xyz="0 0 1" />
-    <limit effort = "1000.0" velocity = "1.0" lower = "-3.14" upper = "3.14"/>
-  </joint>
-  <link
-    name="arm2_tool_link" />
+    <limit effort = "1000.0" velocity = "1.0" lower = "-3.0" upper = "3.0"/>
+  </joint>
+ <link
+    name="arm2_tool_link" >
+  <visual>
+      <origin
+        xyz="0 -0.145 -0.092"
+        rpy="0 0 0" />
+           <!-- <origin
+        xyz="0 0.145 0.0748"
+        rpy="0 0 0" /> -->
+      <geometry>
+          <mesh
+    filename="package://agv_description/meshes/tool.STL"
+    scale="0.001 0.001 0.001" />
+      </geometry>
+    </visual>
+  </link>
   <joint
     name="arm2_tool_joint" type="fixed">
@@ -928,3 +969,12 @@
       <origin xyz="0 0 0.054" rpy="0 0 0" />
   </joint>
+  <link
+    name="arm2_toolscan_link" />
+  <joint
+    name="arm2_toolscan_joint" type="fixed">
+      <parent link="arm2_tool_link" />
+      <child link="arm2_toolscan_link" />
+      <!-- <origin xyz="0 0.2 0.0748" rpy="1.5708 0 0" /> -->
+      <origin xyz="0 -0.18 0.0748" rpy="-1.5708 3.14159 0" />
+  </joint>
 </robot>
